Commit message: add base penalty

File: src/curobo/content/assets/robot/jaka_description/left_jaka_mobile.urdf (robot description, URDF)
Before this commit: robot jaka_mobile, 11 links, 10 joints
Joints:
- joint base_x: limit lower=-0.05 upper=0.05 effort=100 velocity=1.0 -> lower=-0.08 upper=0.08 effort=100 velocity=1.0
- joint base_y: limit lower=-0.05 upper=0.05 effort=100 velocity=1.0 -> lower=-0.08 upper=0.08 effort=100 velocity=1.0
