Commit message: add workspacte anlysis

File: src/curobo/content/assets/robot/jaka_description/left_jaka.urdf (robot description, URDF)
Before this commit: robot jaka, 8 links, 7 joints
Links:
- added link tool
Joints:
- added joint tool_joint: type fixed, parent LINK_7, child tool, origin xyz=0 0 0.14 rpy=0 0 0
- joint J_1: limit lower=-6.1927 upper=6.1927 effort=0 velocity=0 -> lower=-6.196 upper=6.196 effort=0 velocity=0
- joint J_2: limit lower=-1.6572 upper=1.6572 effort=0 velocity=0 -> lower=-1.658 upper=1.658 effort=0 velocity=0
- joint J_3: limit lower=-6.1927 upper=6.1927 effort=0 velocity=0 -> lower=-6.196 upper=6.196 effort=0 velocity=0
- joint J_4: limit lower=-2.2677 upper=0.3837 effort=0 velocity=0 -> lower=-2.269 upper=0.384 effort=0 velocity=0
- joint J_5: limit lower=-6.1927 upper=6.1927 effort=0 velocity=0 -> lower=-6.196 upper=6.196 effort=0 velocity=0
- joint J_6: limit lower=-1.5707 upper=1.5707 effort=0 velocity=0 -> lower=-1.571 upper=1.571 effort=0 velocity=0
- joint J_7: limit lower=-6.1927 upper=6.1927 effort=0 velocity=0 -> lower=-6.196 upper=6.196 effort=0 velocity=0
