Commit message: Add robot assets and XTrainer planning tools

File: src/curobo/content/assets/robot/jaka_description/left_jaka.urdf (robot description, URDF)
Before this commit: robot jaka, 9 links, 8 joints
Links:
- removed link tool
- added link gripper_link
Joints:
- removed joint tool_joint
- added joint gripper_joint: type fixed, parent LINK_7, child gripper_link, origin xyz=0 0 0.14 rpy=0 0 0

File: src/curobo/content/assets/robot/marvin_description/urdf/marvin_robot.urdf (robot description, URDF)
Before this commit: robot Marvin M6-S-CCS-696-V4.0_Robot Stand_Asm, 10 links, 9 joints
Joints:
- joint Fix_Base_L: origin xyz=0 0.037 0.14 rpy=-1.5708 0 0 -> xyz=0 0.087 0.14 rpy=-1.57 0 -0.758
- joint gripper_joint: origin xyz=0 -0.25 0 rpy=1.57 0 0 -> xyz=0 -0.31 0 rpy=1.57 1.57 0
