Commit message: add sphere of marvin_arm

File: marvin_arm/Marvin M6-S-CCS-696-V4.0_Robot Stand_Asm/urdf/Marvin M6-S-CCS-696-V4.0_Robot Stand_Asm.urdf (robot description, URDF)
Before this commit: robot Marvin M6-S-CCS-696-V4.0_Robot Stand_Asm, 17 links, 16 joints
Links:
- removed link Base_R
- removed link Link1_R
- removed link Link2_R
- removed link Link3_R
- removed link Link4_R
- removed link Link5_R
- removed link Link6_R
- removed link Link7_R
- link Base_L: geometry collision mesh filename=../meshes/Base_L.STL; visual mesh filename=../meshes/Base_L.STL
- link Link1_L: geometry collision mesh filename=../meshes/Link1_L.STL; visual mesh filename=../meshes/Link1_L.STL
- link Link2_L: geometry collision mesh filename=../meshes/Link2_L.STL; visual mesh filename=../meshes/Link2_L.STL
- link Link3_L: geometry collision mesh filename=../meshes/Link3_L.STL; visual mesh filename=../meshes/Link3_L.STL
- link Link4_L: geometry collision mesh filename=../meshes/Link4_L.STL; visual mesh filename=../meshes/Link4_L.STL
- link Link5_L: geometry collision mesh filename=../meshes/Link5_L.STL; visual mesh filename=../meshes/Link5_L.STL
- link Link6_L: geometry collision mesh filename=../meshes/Link6_L.STL; visual mesh filename=../meshes/Link6_L.STL
- link Link7_L: geometry collision mesh filename=../meshes/Link7_L.STL; visual mesh filename=../meshes/Link7_L.STL
- link robot_stand: geometry collision mesh filename=../meshes/robot_stand.STL; visual mesh filename=../meshes/robot_stand.STL
Joints:
- removed joint Fix_Base_R
- removed joint Joint1_R
- removed joint Joint2_R
- removed joint Joint3_R
- removed joint Joint4_R
- removed joint Joint5_R
- removed joint Joint6_R
- removed joint Joint7_R

Commit message: update file

File: marvin_arm/Marvin M6-S-CCS-696-V4.0_Robot Stand_Asm/urdf/Marvin M6-S-CCS-696-V4.0_Robot Stand_Asm.urdf (robot description, URDF)
Before this commit: robot Marvin M6-S-CCS-696-V4.0_Robot Stand_Asm, 9 links, 8 joints
Links:
- added link gripper_link
Joints:
- added joint gripper_joint: type fixed, parent Link7_L, child gripper_link, origin xyz=0 -0.25 0 rpy=1.57 0 0

File: src/curobo/content/assets/robot/marvin_description/urdf/marvin_robot.urdf (robot description, URDF)
Before this commit: robot Marvin M6-S-CCS-696-V4.0_Robot Stand_Asm, 9 links, 8 joints
Links:
- added link gripper_link
Joints:
- added joint gripper_joint: type fixed, parent Link7_L, child gripper_link, origin xyz=0 -0.25 0 rpy=1.57 0 0
